File: keyboard-project/keyboard-project.kicad_sch (KiCad schematic)
At the start: 0 parts

Commit message: Create sheets for each subsystem
Other:
- added sheet BLE (ble.kicad_sch)
- added sheet Display (display.kicad_sch)
- added sheet Encoders (encoders.kicad_sch)
- added sheet Key Matrix (key_matrix.kicad_sch)
- added sheet LED (led.kicad_sch)
- added sheet MCU (mcu.kicad_sch)
- added sheet Power (power.kicad_sch)
- added sheet Trackball (trackball.kicad_sch)
- added sheet USB (usb.kicad_sch)
- note added: "1"
- note added: "5/3/26"
- note added: "Block Diagram"
