File: keyboard-project/ble.kicad_sch (KiCad schematic)
At the start: 0 parts

Commit message: ble update
Parts:
- added C32, C33: C, symbol Device:C
- added J4: Conn_01x04_Pin, symbol Connector:Conn_01x04_Pin
- added R10: 0, symbol Device:R_US
- added U6: HOLYIOT-18010-NRF52840, HOLYIOT-18010-NRF52840:XCVR_HOLYIOT-18010-NRF52840, symbol HOLYIOT-18010-NRF52840:HOLYIOT-18010-NRF52840
Connections:
- new net: R10.2, U6.21 (P0_18)
- new net: J4.3 (Pin_3), U6.32 (SWDIO)
- new net: J4.4 (Pin_4), U6.31 (SWDCLK)
- new net +3.3VA: C32.1, C33.1, J4.1 (Pin_1), U6.14 (VDD_NRF)
- new net GND: C32.2, C33.2, J4.2 (Pin_2), U6.1 (GND), U6.25 (GND), U6.37 (GND)
- new net USART1_RX: U6.45 (P0_06)
- new net USART1_TX: U6.44 (P0_08)
- new net nRF52840 RST: R10.1
- new net nRF52840 WAKE: U6.41 (P0_11)
- no-connect marks 0 -> 45
Other:
- note added: "25, 37 to GND"
- note added: "5/7/26"
- note added: "BLE Module"
- note added: "Bridge, remove after board is flashed."
- note added: "Debug header"

Commit message: res and cap footprints
Parts:
- C32, C33: footprint (none) -> Capacitor_SMD:C_1206_3216Metric_Pad1.33x1.80mm_HandSolder
- R10: footprint (none) -> Resistor_SMD:R_1206_3216Metric_Pad1.30x1.75mm_HandSolder
Other:
- note added: "BLE Debug header"
- note removed: "Debug header"
Changed lines of the file:
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@@
 		)
 	)
-	(text "Debug header"
+	(text "BLE Debug header"
 		(exclude_from_sim no)
-		(at 260.604 79.756 0)
+		(at 257.556 80.01 0)
 		(effects
 			(font
@@
 			)
 		)
-		(property "Footprint" ""
+		(property "Footprint" "Capacitor_SMD:C_1206_3216Metric_Pad1.33x1.80mm_HandSolder"
 			(at 204.1652 58.42 0)
 			(hide yes)
@@
 			)
 		)
-		(property "Footprint" ""
+		(property "Footprint" "Capacitor_SMD:C_1206_3216Metric_Pad1.33x1.80mm_HandSolder"
 			(at 191.4652 58.42 0)
 			(hide yes)
@@
 			)
 		)
-		(property "Footprint" ""
+		(property "Footprint" "Resistor_SMD:R_1206_3216Metric_Pad1.30x1.75mm_HandSolder"
 			(at 99.314 92.964 90)
 			(hide yes)

Commit message: all footprints in now
Parts:
- J4: footprint (none) -> Connector_JST:JST_EH_B4B-EH-A_1x04_P2.50mm_Vertical
- U6: footprint HOLYIOT-18010-NRF52840:XCVR_HOLYIOT-18010-NRF52840 -> kicad-footprints:XCVR_HOLYIOT-18010-NRF52840
Changed lines of the file:
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@@
 			)
 		)
-		(property "Footprint" ""
+		(property "Footprint" "Connector_JST:JST_EH_B4B-EH-A_1x04_P2.50mm_Vertical"
 			(at 259.08 73.66 0)
 			(hide yes)
@@
 			)
 		)
-		(property "Footprint" "HOLYIOT-18010-NRF52840:XCVR_HOLYIOT-18010-NRF52840"
+		(property "Footprint" "kicad-footprints:XCVR_HOLYIOT-18010-NRF52840"
 			(at 148.59 88.9 0)
 			(hide yes)
