File: keyboard-project/usb.kicad_sch (KiCad schematic)
At the start: 0 parts

Commit message: ble update
Parts:
- added C31: 100n, symbol Device:C
- added FB1, FB2: 600 @ 100MHz, symbol Device:FerriteBead
- added J3: USB_C_Receptacle, symbol Connector:USB_C_Receptacle
- added R13, R14: R_US, symbol Device:R_US
- added R6, R9: 5.1k, symbol Device:R_US
Connections:
- new net: J3.A5 (CC1), R6.1
- new net: FB2.1, J3.A6 (D+), J3.B6 (D+)
- new net: FB1.1, J3.A7 (D-), J3.B7 (D-)
- new net: J3.B5 (CC2), R9.1
- new net +5V: C31.2, J3.A4 (VBUS), J3.A9 (VBUS), J3.B4 (VBUS), J3.B9 (VBUS), R13.1
- new net GND: C31.1, J3.A1 (GND), J3.A12 (GND), J3.B1 (GND), J3.B12 (GND), J3.SH (SHIELD), R14.2, R6.2, R9.2
- new net USB D+: FB2.2
- new net USB D-: FB1.2
- new net VBUS Detect: R13.2, R14.1
- no-connect marks 0 -> 10
Other:
- note added: "5/3/26"
- note added: "VBUS detection on the MCU, should ouput 2V5 when USB is plugged in"

Commit message: res and cap footprints
Parts:
- C31: footprint (none) -> Capacitor_SMD:C_1206_3216Metric_Pad1.33x1.80mm_HandSolder
- R6, R9: footprint (none) -> Resistor_SMD:R_1206_3216Metric_Pad1.30x1.75mm_HandSolder
Changed lines of the file:
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@@
 			)
 		)
-		(property "Footprint" ""
+		(property "Footprint" "Resistor_SMD:R_1206_3216Metric_Pad1.30x1.75mm_HandSolder"
 			(at 103.124 71.374 90)
 			(hide yes)
@@
 			)
 		)
-		(property "Footprint" ""
+		(property "Footprint" "Capacitor_SMD:C_1206_3216Metric_Pad1.33x1.80mm_HandSolder"
 			(at 95.25 48.5648 0)
 			(hide yes)
@@
 			)
 		)
-		(property "Footprint" ""
+		(property "Footprint" "Resistor_SMD:R_1206_3216Metric_Pad1.30x1.75mm_HandSolder"
 			(at 118.364 73.914 90)
 			(hide yes)

Commit message: more footprints
Parts:
- FB1, FB2: footprint (none) -> Inductor_SMD:L_Walsin_WLFM201209x
- J3: footprint (none) -> Connector_USB:USB_C_Receptacle_GCT_USB4105-xx-A_16P_TopMnt_Horizontal
Changed lines of the file:
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@@
 			)
 		)
-		(property "Footprint" ""
+		(property "Footprint" "Connector_USB:USB_C_Receptacle_GCT_USB4105-xx-A_16P_TopMnt_Horizontal"
 			(at 83.82 92.71 0)
 			(hide yes)
@@
 			)
 		)
-		(property "Footprint" ""
+		(property "Footprint" "Inductor_SMD:L_Walsin_WLFM201209x"
 			(at 167.64 88.138 90)
 			(hide yes)
@@
 			)
 		)
-		(property "Footprint" ""
+		(property "Footprint" "Inductor_SMD:L_Walsin_WLFM201209x"
 			(at 135.89 83.058 90)
 			(hide yes)

Commit message: all footprints in now
Parts:
- R13, R14: footprint (none) -> Resistor_SMD:R_1206_3216Metric_Pad1.30x1.75mm_HandSolder
Changed lines of the file:
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@@
 			)
 		)
-		(property "Footprint" ""
+		(property "Footprint" "Resistor_SMD:R_1206_3216Metric_Pad1.30x1.75mm_HandSolder"
 			(at 22.606 39.624 90)
 			(hide yes)
@@
 			)
 		)
-		(property "Footprint" ""
+		(property "Footprint" "Resistor_SMD:R_1206_3216Metric_Pad1.30x1.75mm_HandSolder"
 			(at 22.606 26.924 90)
 			(hide yes)
