File: keyboard-project/power.kicad_sch (KiCad schematic)
At the start: 23 parts, among them J1 Conn_01x02, U1 MCP1826S, U2 MCP73871, U3 XC6206PxxxMR, U4 AP7331-28WG-7

Commit message: more footprints
Changed lines of the file:
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@@
+	(polyline
+		(pts
+			(xy 72.39 67.31) (xy 72.39 68.58)
+		)
+		(stroke
+			(width 0)
+			(type default)
+		)
+	)
 	(polyline
 		(pts
