File: keyboard-project/keyboard-project.kicad_pcb (KiCad board)
At the start: 6 copper layers, 460 x 140 mm, 389 parts, among them J1 Conn_01x02, J2 TC2030, J3 USB_C_Receptacle, J4 Conn_01x04_Pin, J5 Conn_01x14_Pin, SW1 SW_Push, SW10 SW_Push, SW103 RotaryEncoder_Switch_MP, SW104 RotaryEncoder_Switch_MP, SW105 RotaryEncoder_Switch_MP, SW11 SW_Push, SW12 SW_Push, SW13 SW_Push, SW14 SW_Push, SW15 SW_Push, SW16 SW_Push, SW17 SW_Push, SW18 SW_Push, SW19 SW_Push, SW2 SW_Push, SW20 SW_Push, SW21 SW_Push, SW22 SW_Push, SW23 SW_Push, SW24 SW_Push, SW25 SW_Push, SW26 SW_Push, SW27 SW_Push, SW28 SW_Push, SW29 SW_Push, SW3 SW_Push, SW30 SW_Push, SW31 SW_Push, SW32 SW_Push, SW33 SW_Push, SW34 SW_Push, SW35 SW_Push, SW36 SW_Push, SW37 SW_Push, SW38 SW_Push, SW39 SW_Push, SW4 SW_Push, SW40 SW_Push, SW41 SW_Push, SW42 SW_Push, SW43 SW_Push, SW44 SW_Push, SW45 SW_Push, SW46 SW_Push, SW47 SW_Push, SW48 SW_Push, SW49 SW_Push, SW5 SW_Push, SW50 SW_Push, SW51 SW_Push, SW52 SW_Push, SW53 SW_Push, SW54 SW_Push, SW55 SW_Push, SW56 SW_Push, SW57 SW_Push, SW58 SW_Push, SW59 SW_Push, SW6 SW_Push, SW60 SW_Push, SW61 SW_Push, SW62 SW_Push, SW63 SW_Push, SW64 SW_Push, SW65 SW_Push, SW66 SW_Push, SW67 SW_Push, SW68 SW_Push, SW69 SW_Push, SW7 SW_Push, SW70 SW_Push, SW71 SW_Push, SW72 SW_Push, SW73 SW_Push, SW74 SW_Push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

Commit message: more footprints
Parts:
- C31, C32, C33, FB1, FB2, J1, J2, J4, R10, R13, R14, R6, R9, U6, U8: moved to B.Cu
- moved U7 396.5 mm to (499.1, 62.3)
- moved R14 393.0 mm to (446.5, 58.5)
- moved R13 386.7 mm to (439.4, 58.5)
- moved C31 379.1 mm to (424.4, 59.5)
- moved R9 378.5 mm to (433.1, 61.0)
- moved FB2 376.4 mm to (431.0, 65.5), turned to -90 degrees
- moved FB1 372.6 mm to (428.0, 65.5), turned to -90 degrees
- moved R6 370.7 mm to (424.4, 62.0), turned to 180 degrees
- moved R10 349.8 mm to (93.5, 59.0)
- moved C33 343.5 mm to (92.0, 64.5), turned to 90 degrees
- moved C32 338.7 mm to (95.5, 64.5), turned to 90 degrees
- moved U6 333.9 mm to (108.0, 63.0), turned to 90 degrees
- moved J1 324.8 mm to (449.5, 81.5), turned to 180 degrees
- moved J4 323.7 mm to (387.5, 55.0), turned to 180 degrees
- moved SW104 321.2 mm to (504.9, 95.0), turned to 180 degrees
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Routing:
- net GND: track 96.8 -> 128.6 mm
- net +3.3VA: track 2.91 -> 18.2 mm
- net +5V: track 3.21 -> 15.5 mm, vias 0 -> 3
- net Net-(FB2-Pad1): track 2.44 -> 10.6 mm
- net Net-(FB1-Pad1): track 2.44 -> 10.6 mm
- net Net-(J3-CC1): track 0.00 -> 7.04 mm
- net Net-(U6-P0_18): track 0.00 -> 5.05 mm
- net Net-(J3-CC2): track 0.00 -> 4.42 mm
- net VBUS Detect: track 0.00 -> 3.95 mm, vias 0 -> 1
Other:
- board text added: "2V Regulator"
- board text added: "3V3 Regulator"
- board text added: "3V3, GND, IO, CLK"
- board text added: "BLE Debug"
- board text added: "BLE Module"
- board text added: "Battery Charge Controller"
- board text added: "GND, X, 3V3 NRST, IO, CLK"
- board text added: "MCU Debug"
- board text added: "Playback"
- board text added: "Scroll"
- board text added: "Volume"

Commit message: pcb layout - keys and diodes
Parts:
- D1, D10, D100, D11, D12, D13, D14, D15, D17, D18, D19, D20, D21, D22, D23, D24, D25, D26, D27, D28, D29, D30, D31, D32, D33, D34, D35, D36, D37, D38, D39, D4, D40, D41, D42, D43, D44, D45, D46, D47, D48, D49, D5, D50, D51, D52, D53, D54, D55, D56, D57, D58, D59, D6, D60, D61, D62, D63, D65, D67, D69, D7, D71, D72, D73, D74, D75, D76, D77, D79, D8, D81, D82, D83, D85, D87, D88, D89, D9, D90, D91, D92, D93, D94, D95, D96, D97, D98, D99: moved to B.Cu
- moved C32 415.0 mm to (411.2, 333.9)
- moved C33 415.0 mm to (407.7, 333.9)
- moved C4 415.0 mm to (407.2, 344.4)
- moved C5 415.0 mm to (401.7, 339.9)
- moved R10 415.0 mm to (409.2, 328.4)
- moved U3 415.0 mm to (405.7, 339.4)
- moved U6 415.0 mm to (423.7, 332.4)
- moved SW33 391.0 mm to (406.0, 86.0)
- moved SW32 366.9 mm to (386.9, 86.0)
- moved U8 366.1 mm to (468.6, 291.6)
- moved SW16 366.1 mm to (406.0, 67.0)
- moved SW11 350.8 mm to (265.5, 67.0)
- moved SW31 342.7 mm to (367.9, 86.0)
- moved SW15 341.8 mm to (386.9, 67.0)
- moved SW10 328.5 mm to (246.4, 67.0)
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Routing:
- net CHARGER OUT / REGULATOR IN: track 490.2 -> 131.9 mm
- net Matrix Row 1: track 0.00 -> 333.7 mm
- net Matrix Row 0: track 0.00 -> 331.0 mm
- net Matrix Row 5: track 0.00 -> 331.0 mm
- net Matrix Row 2: track 0.00 -> 326.2 mm
- net Matrix Row 4: track 0.00 -> 304.4 mm
- net Matrix Row 3: track 0.00 -> 249.2 mm
- net Matrix Col 11: track 0.00 -> 124.3 mm
- net Matrix Col 10: track 0.00 -> 123.1 mm
- net Matrix Col 1: track 0.00 -> 122.4 mm
- net Matrix Col 9: track 0.00 -> 118.1 mm
- net Matrix Col 8: track 0.00 -> 113.5 mm
- net Matrix Col 2: track 0.00 -> 113.5 mm
- net Matrix Col 0: track 0.00 -> 111.6 mm
- net Matrix Col 5: track 0.00 -> 110.8 mm
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- removed copper zone on In3.Cu, net +3.3V
- removed copper zone on In2.Cu, net GND
Other:
- board text added: "-"
- board text added: "0"
- board text added: "1"
- board text added: "2"
- board text added: "3"
- board text added: "4"
- board text added: "5"
- board text added: "6"
- board text added: "7"
- board text added: "8"
- board text added: "9"
- board text added: ";"
- board text added: "<"
- board text added: "="
- board text added: ">"
- board text added: "?"
- board text added: "A"
- board text added: "B"
- board text added: "BKSP"
- board text added: "C"
- board text added: "CAPS"
- board text added: "CNTXT"
- board text added: "D"
- board text added: "DEL"
- board text added: "E"
- board text added: "END"
- board text added: "ENTR"
- board text added: "ESC"
- board text added: "F"
- board text added: "F1"
- board text added: "F10"
- board text added: "F11"
- board text added: "F12"
- board text added: "F2"
- board text added: "F3"
- board text added: "F4"
- board text added: "F5"
- board text added: "F6"
- board text added: "F7"
- board text added: "F8"
- board text added: "F9"
- board text added: "G"
- board text added: "H"
- board text added: "HME"
- board text added: "I"
- board text added: "INS"
- board text added: "J"
- board text added: "K"
- board text added: "L"
- board text added: "L ALT"
- board text added: "L CTRL"
- board text added: "L SHFT"
- board text added: "L SUP"
- board text added: "M"
- board text added: "N"
- board text added: "O"
- board text added: "P"
- board text added: "PG DWN"
- board text added: "PG UP"
- board text added: "PRNT"
- board text added: "PSE"
- board text added: "Q"
- board text added: "R"
- board text added: "R ALT"
- board text added: "R CTRL"
- board text added: "R SHFT"
- board text added: "R SUP"
- board text added: "S"
- board text added: "SCL LCK"
- board text added: "SPC"
- board text added: "T"
- board text added: "TAB"
- board text added: "U"
- board text added: "V"
- board text added: "W"
- board text added: "X"
- board text added: "Y"
- board text added: "Z"
- board text added: "["
- board text added: "]"
- board text added: "{dblquote}"
- board text added: "|"
- board text added: "~"

Commit message: pcb layout, leds for keycaps
Parts:
- moved D118 227.2 mm to (365.3, 76.3)
- moved D121 226.7 mm to (72.5, 95.4)
- moved D138 224.5 mm to (77.2, 114.4)
- moved D155 224.3 mm to (79.6, 133.5)
- moved D105 220.3 mm to (72.5, 76.3)
- moved D181 219.5 mm to (74.8, 171.6)
- moved D106 216.2 mm to (91.5, 76.3)
- moved D122 214.1 mm to (91.5, 95.4)
- moved D168 214.1 mm to (84.3, 152.5)
- moved D139 207.7 mm to (101.1, 114.4)
- moved D107 205.6 mm to (110.6, 76.3)
- moved D120 205.1 mm to (403.4, 76.3)
- moved D156 205.1 mm to (105.8, 133.5)
- moved D123 202.6 mm to (110.6, 95.4)
- moved D117 198.8 mm to (301.1, 76.3)
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Routing:
- net SW2: track 0.00 -> 711.9 mm, vias 0 -> 10
- net SW1: track 0.00 -> 515.8 mm, vias 0 -> 10
- net CS22: track 0.00 -> 328.7 mm, vias 0 -> 9
- net CS24: track 0.00 -> 324.2 mm, vias 0 -> 9
- net CS23: track 0.00 -> 324.2 mm, vias 0 -> 9
- net CS31: track 0.00 -> 197.3 mm, vias 0 -> 9
- net CS32: track 0.00 -> 195.6 mm, vias 0 -> 9
- net CS33: track 0.00 -> 195.6 mm, vias 0 -> 9
- net CS19: track 0.00 -> 183.6 mm, vias 0 -> 9
- net CS7: track 0.00 -> 183.5 mm, vias 0 -> 9
- net CS16: track 0.00 -> 183.4 mm, vias 0 -> 9
- net CS20: track 0.00 -> 181.9 mm, vias 0 -> 9
- net CS21: track 0.00 -> 181.9 mm, vias 0 -> 9
- net CS18: track 0.00 -> 181.9 mm, vias 0 -> 9
- net CS17: track 0.00 -> 181.9 mm, vias 0 -> 9
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
Commit message: more layout, all keycaps/leds are routed, need to place ICs now
Parts:
- SW84: moved to B.Cu
- moved J5 346.8 mm to (532.6, 133.8)
- moved C32 276.7 mm to (495.4, 70.3)
- moved C33 276.7 mm to (491.9, 70.3)
- moved C4 276.7 mm to (491.4, 80.8)
- moved C5 276.7 mm to (485.9, 76.3)
- moved R10 276.7 mm to (493.4, 64.8)
- moved U3 276.7 mm to (489.9, 75.8)
- moved U6 276.7 mm to (507.9, 68.8)
- moved C2 199.9 mm to (428.0, 117.8)
- moved C3 199.9 mm to (428.0, 131.8)
- moved U1 199.9 mm to (425.0, 125.0)
- moved U8 185.1 mm to (384.4, 126.8)
- moved C1 180.2 mm to (456.4, 102.4)
- moved R1 180.2 mm to (448.9, 96.9)
- moved R2 180.2 mm to (448.9, 88.9)
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Routing:
- net SW9: track 15.4 -> 776.8 mm, vias 9 -> 11
- net SW7: track 14.9 -> 756.5 mm, vias 9 -> 11
- net SW3: track 17.3 -> 724.3 mm, vias 10 -> 13
- net SW5: track 16.6 -> 683.3 mm, vias 10 -> 14
- net SW6: track 16.6 -> 678.8 mm, vias 10 -> 13
- net SW8: track 14.9 -> 658.7 mm, vias 9 -> 11
- net SW4: track 16.6 -> 577.7 mm, vias 10 -> 13
- net SW1: track 515.8 -> 701.8 mm, vias 10 -> 14
- net GND: track 128.6 -> 111.3 mm, vias 4 -> 3
- net SW2: track 711.9 -> 703.9 mm, vias 10 -> 13
- net BAT +: track 4.40 -> 6.42 mm
- net Matrix Row 4: track 304.4 -> 302.7 mm
- net Matrix Col 3: track 90.0 -> 90.8 mm
- net Matrix Col 2: track 113.5 -> 114.0 mm
- net +3.3V: vias 3 -> 2
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
Commit message: resistors and caps for mcu
Parts:
- C10, C11, C12, C13, C14, C15, C16, C17, C18, C19, C20, C21, C22, C23, C24, C25, C26, C27, C28, C29, C30, C34, C35, C36, C9, R15, R16, R17, R18, R19, R20, R21, R22, R23, R24, R25, R26, R27, R28, R29, R30, R31: moved to B.Cu
- moved SW104 537.0 mm to (43.4, 98.7), turned to -90 degrees
- moved SW105 536.2 mm to (43.4, 123.0), turned to -90 degrees
- moved U6 483.6 mm to (34.8, 168.6), turned to -90 degrees
- moved C6 460.1 mm to (49.8, 142.6)
- moved C7 460.1 mm to (52.8, 142.6)
- moved U4 460.1 mm to (51.3, 137.6)
- moved C32 458.5 mm to (47.2, 167.1), turned to -90 degrees
- moved R10 456.9 mm to (49.3, 172.6), turned to 180 degrees
- moved C33 451.6 mm to (50.8, 167.1), turned to -90 degrees
- moved C4 446.6 mm to (51.2, 156.6), turned to 90 degrees
- moved U3 445.5 mm to (52.8, 161.6), turned to 180 degrees
- moved C5 437.4 mm to (56.8, 161.1), turned to 90 degrees
- moved J4 371.5 mm to (90.0, 221.1)
- moved D97 344.8 mm to (31.0, 65.3), turned to -90 degrees
- moved D96 324.2 mm to (50.0, 65.3), turned to -90 degrees
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Routing:
- net Matrix Row 5: track 331.0 -> 464.3 mm, vias 0 -> 2
- net CHARGER OUT / REGULATOR IN: track 131.9 -> 21.5 mm
- net Matrix Row 0: track 331.0 -> 228.6 mm
- net I2C1_SCL: track 0.00 -> 34.8 mm
- net I2C1_SDA: track 0.00 -> 34.7 mm
- net GND: track 111.3 -> 135.3 mm, vias 3 -> 5
- net Net-(D3-K): track 60.7 -> 78.9 mm
- net Net-(D2-K): track 57.2 -> 72.5 mm, vias 1 -> 2
- net ENC 3 PHASE B: track 0.00 -> 11.8 mm
- net NRST: track 0.00 -> 10.5 mm
- net ENC 3 PHASE A: track 0.00 -> 10.2 mm
- net Net-(C19-Pad1): track 0.00 -> 9.23 mm
- net +3.3V: track 15.3 -> 7.86 mm, vias 2 -> 3
- net Net-(C25-Pad1): track 0.00 -> 7.22 mm
- net Net-(C29-Pad1): track 0.00 -> 7.02 mm
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- added copper zone on In5.Cu, net +3.3V
- added copper zone on In6.Cu, net GND
Other:
- board size 460 x 140 mm -> 500 x 120 mm
- copper layers 6 -> 8
- board text added: "3V3A, GND, IO, CLK"
- board text removed: "3V3, GND, IO, CLK"
